Commit message: feat: drive wheels and caster spheres using parametrized macros)

File: ws/src/helmsman_description/urdf/helmsman.urdf.xacro (robot description, xacro)
@@ -8,4 +8,11 @@
     <xacro:property name="wheel_radius" value="0.085"/>
     <xacro:property name="ground_clearance" value="0.04"/>
+    <xacro:property name="wheel_width" value="0.04"/>
+    <xacro:property name="wheel_mass" value="1.5"/>
+    <xacro:property name="wheel_x_offset" value="0.0"/>
+    <xacro:property name="caster_radius" value="0.04"/>
+    <xacro:property name="caster_mass" value="0.3"/>
+    <xacro:property name="caster_x" value="0.30"/>
+    <xacro:property name="caster_y" value="0.17"/>
     <!-- ================= Materials (as macros, inlined per visual) ================= -->
     <xacro:macro name="mat_charcoal">
@@ -41,4 +48,77 @@
         </inertial>
     </xacro:macro>
+    <xacro:macro name="cylinder_inertia" params="m r h">
+        <inertial>
+            <mass value="${m}"/>
+            <inertia ixx="${(m/12.0)*(3*r*r + h*h)}" ixy="0" ixz="0" iyy="${(m/12.0)*(3*r*r + h*h)}" iyz="0" izz="${(m/2.0)*r*r}"/>
+        </inertial>
+    </xacro:macro>
+    <xacro:macro name="sphere_inertia" params="m r">
+        <inertial>
+            <mass value="${m}"/>
+            <inertia ixx="${(2.0/5.0)*m*r*r}" ixy="0" ixz="0" iyy="${(2.0/5.0)*m*r*r}" iyz="0" izz="${(2.0/5.0)*m*r*r}"/>
+        </inertial>
+    </xacro:macro>
+    <!-- ================= Drive wheels ================= -->
+    <xacro:macro name="drive_wheel" params="side reflect">
+        <link name="${side}_wheel_link">
+            <visual>
+                <origin rpy="${pi/2} 0 0"/>
+                <geometry>
+                    <cylinder radius="${wheel_radius}" length="${wheel_width}"/>
+                </geometry>
+                <xacro:mat_charcoal/>
+            </visual>
+            <!-- hub cap: shallower, slightly wider-looking dark disc -->
+            <visual>
+                <origin xyz="0 ${reflect * wheel_width/2} 0" rpy="${pi/2} 0 0"/>
+                <geometry>
+                    <cylinder radius="${wheel_radius * 0.55}" length="0.005"/>
+                </geometry>
+                <xacro:mat_dark_gray/>
+            </visual>
+            <collision>
+                <origin rpy="${pi/2} 0 0"/>
+                <geometry>
+                    <cylinder radius="${wheel_radius}" length="${wheel_width}"/>
+                </geometry>
+            </collision>
+            <xacro:cylinder_inertia m="${wheel_mass}" r="${wheel_radius}" h="${wheel_width}"/>
+        </link>
+        <joint name="${side}_wheel_joint" type="continuous">
+            <parent link="base_link"/>
+            <child link="${side}_wheel_link"/>
+            <origin xyz="${wheel_x_offset} ${reflect * (body_width/2 + wheel_width/2 + 0.005)} ${-(ground_clearance + body_height/2) + wheel_radius}" rpy="0 0 0"/>
+            <axis xyz="0 1 0"/>
+        </joint>
+    </xacro:macro>
+    <xacro:drive_wheel side="left" reflect="1"/>
+    <xacro:drive_wheel side="right" reflect="-1"/>
+    <!-- ================= Casters: frictionless spheres ================= -->
+    <xacro:macro name="caster" params="prefix x_reflect y_reflect">
+        <link name="${prefix}_caster_link">
+            <visual>
+                <geometry>
+                    <sphere radius="${caster_radius}"/>
+                </geometry>
+                <xacro:mat_dark_gray/>
+            </visual>
+            <collision>
+                <geometry>
+                    <sphere radius="${caster_radius}"/>
+                </geometry>
+            </collision>
+            <xacro:sphere_inertia m="${caster_mass}" r="${caster_radius}"/>
+        </link>
+        <joint name="${prefix}_caster_joint" type="fixed">
+            <parent link="base_link"/>
+            <child link="${prefix}_caster_link"/>
+            <origin xyz="${x_reflect * caster_x} ${y_reflect * caster_y} ${-(ground_clearance + body_height/2) + caster_radius}"/>
+        </joint>
+    </xacro:macro>
+    <xacro:caster prefix="front_left" x_reflect="1" y_reflect="1"/>
+    <xacro:caster prefix="front_right" x_reflect="1" y_reflect="-1"/>
+    <xacro:caster prefix="rear_left" x_reflect="-1" y_reflect="1"/>
+    <xacro:caster prefix="rear_right" x_reflect="-1" y_reflect="-1"/>
     <!-- ================= base_footprint ================= -->
     <link name="base_footprint"/>

Commit message: feat: lidar and tilted depth camera with optical frame

File: ws/src/helmsman_description/urdf/helmsman.urdf.xacro (robot description, xacro)
@@ -15,4 +15,10 @@
     <xacro:property name="caster_x" value="0.30"/>
     <xacro:property name="caster_y" value="0.17"/>
+    <xacro:property name="mast_height" value="0.18"/>
+    <xacro:property name="mast_radius" value="0.02"/>
+    <xacro:property name="lidar_radius" value="0.05"/>
+    <xacro:property name="lidar_height" value="0.05"/>
+    <xacro:property name="lidar_mass" value="0.4"/>
+    <xacro:property name="camera_tilt_deg" value="12"/>
     <!-- ================= Materials (as macros, inlined per visual) ================= -->
     <xacro:macro name="mat_charcoal">
@@ -183,4 +189,12 @@
             <xacro:mat_orange/>
         </visual>
+        <!-- sensor mast, rear of deck -->
+        <visual>
+            <origin xyz="-0.25 0 ${body_height/2 + 0.02 + mast_height/2}"/>
+            <geometry>
+                <cylinder radius="${mast_radius}" length="${mast_height}"/>
+            </geometry>
+            <xacro:mat_light_gray/>
+        </visual>
         <!-- ONE simple collision for the whole chassis -->
         <collision>
@@ -191,3 +205,65 @@
         <xacro:box_inertia m="${body_mass}" x="${body_length}" y="${body_width}" z="${body_height}"/>
     </link>
+    <!-- ================= Lidar ================= -->
+    <link name="lidar_link">
+        <visual>
+            <geometry>
+                <cylinder radius="${lidar_radius}" length="${lidar_height}"/>
+            </geometry>
+            <xacro:mat_charcoal/>
+        </visual>
+        <!-- emitter window band -->
+        <visual>
+            <origin xyz="0 0 0.005"/>
+            <geometry>
+                <cylinder radius="${lidar_radius + 0.002}" length="0.012"/>
+            </geometry>
+            <xacro:mat_teal/>
+        </visual>
+        <collision>
+            <geometry>
+                <cylinder radius="${lidar_radius}" length="${lidar_height}"/>
+            </geometry>
+        </collision>
+        <xacro:cylinder_inertia m="${lidar_mass}" r="${lidar_radius}" h="${lidar_height}"/>
+    </link>
+    <joint name="lidar_joint" type="fixed">
+        <parent link="base_link"/>
+        <child link="lidar_link"/>
+        <origin xyz="-0.25 0 ${body_height/2 + 0.02 + mast_height + lidar_height/2}" rpy="0 0 0"/>
+    </joint>
+    <!-- ================= Depth camera ================= -->
+    <link name="camera_link">
+        <visual>
+            <geometry>
+                <box size="0.02 0.09 0.025"/>
+            </geometry>
+            <xacro:mat_charcoal/>
+        </visual>
+        <!-- lens dot -->
+        <visual>
+            <origin xyz="0.011 0 0" rpy="0 ${pi/2} 0"/>
+            <geometry>
+                <cylinder radius="0.008" length="0.004"/>
+            </geometry>
+            <xacro:mat_teal/>
+        </visual>
+        <collision>
+            <geometry>
+                <box size="0.02 0.09 0.025"/>
+            </geometry>
+        </collision>
+        <xacro:box_inertia m="0.1" x="0.02" y="0.09" z="0.025"/>
+    </link>
+    <joint name="camera_joint" type="fixed">
+        <parent link="base_link"/>
+        <child link="camera_link"/>
+        <origin xyz="${body_length/2 - 0.005} 0 ${body_height/2 - 0.02}" rpy="0 ${camera_tilt_deg * pi / 180.0} 0"/>
+    </joint>
+    <link name="camera_optical_frame"/>
+    <joint name="camera_optical_joint" type="fixed">
+        <parent link="camera_link"/>
+        <child link="camera_optical_frame"/>
+        <origin xyz="0 0 0" rpy="${-pi/2} 0 ${-pi/2}"/>
+    </joint>
 </robot>
